File: stm32f103c8tx_breakout.kicad_pcb (KiCad board)
At the start: 2 copper layers, 45.7 x 45.7 mm, 33 parts, among them J1 USB_B_Micro, J2 Conn_02x05_Odd_Even, J3 Conn_01x12, J4 Conn_01x07, J5 Conn_01x12, J6 Conn_01x06, SW1 SW_SPDT, U1 AMS1117-3.3, U2 STM32F103C8T6, Y1 16M

Commit message: Changed routing to use 4 layers, with internal gnd and 3v3 planes
Parts:
- moved C12 3.07 mm to (37.5, 40.4), turned to 0 degrees
- moved C13 2.58 mm to (37.5, 46.0), turned to 180 degrees
- moved R1 1.78 mm to (58.2, 41.9)
- moved C4 1.14 mm to (55.6, 39.6)
- moved C6 1.00 mm to (45.7, 38.1), turned to 0 degrees
- moved C9 0.23 mm to (43.2, 45.0)
- moved Y1 0.20 mm to (37.5, 43.2)
- moved C8 0.18 mm to (52.1, 49.5)
- moved C5 0.13 mm to (43.2, 39.9), turned to 180 degrees
Routing:
- net +3V3: track 120.8 -> 19.5 mm, vias 2 -> 12
- net PA9: track 29.3 -> 22.4 mm, vias 2 -> 0
- net PA10: track 29.5 -> 22.7 mm, vias 2 -> 0
- net GND: track 34.9 -> 28.1 mm, vias 19 -> 18
- net PA8: track 29.2 -> 22.8 mm
- net NRST: track 20.5 -> 26.6 mm
- net PB14: track 31.4 -> 25.8 mm
- net PB13: track 31.9 -> 27.7 mm
- net PB15: track 27.4 -> 24.1 mm
- net PA1: track 27.5 -> 24.2 mm
- net HSE_IN: track 8.84 -> 11.2 mm
- net PA0: track 26.3 -> 24.4 mm
- net SWDIO: track 21.1 -> 19.2 mm
- net PB12: track 31.0 -> 29.4 mm
- net Net-(C13-Pad1): track 2.79 -> 4.40 mm
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- added copper zone on In2.Cu, net +3V3
- added copper zone on In1.Cu, net GND
- removed copper zone on B.Cu, net GND
Other:
- copper layers 2 -> 4
